File: CAD/TL-WR703N.brd (EAGLE design)
At the start: 48.5 x 50.1 mm, 241 parts, among them T1 H1601CG, U1 AR9331-AL1A, U2 A3S56F40FTP

Commit message: Saved board before linking to schematic
Parts:
- AN1: value (none) -> WIFI_ANTENNA
- D1, D2: value (none) -> MMBD7000
- E$1, E$2, E$3, E$4, E$5, E$6: value (none) -> FIDUCIAL
- E$7: value (none) -> CC-BY-SA
- E$9: value (none) -> GND_3CONTACTS
- GND: value (none) -> TEST_PAD_SHIELD
- J1: value (none) -> JUMPER
- J3: value (none) -> RJ45_2SH
- SW2: value (none) -> TACT_SWITCH_SPST
- T1: value H1601CG -> ETH10_100_TRANSFO
- TP1V2, TP2V0, TP2V5, TP3V3, TPDDR, TPGND, TP_IN, TP_OUT: value (none) -> TEST_PAD
- U5: value (none) -> UNKNOWN_BUCK
- U6: value (none) -> TPS2041BDBV
- USB1: value (none) -> USB-MICROB
- USB2: value (none) -> USB-A_TH
Other:
- outline, holes or cut-outs redrawn

Commit message: Added schematic & update all other files
Parts:
- C1, C17: value (none) -> 1n
- C10, C101, C102, C11, C12, C13, C14, C15, C2, C47, C63, C64, C65, C66, C67, C70, C71, C72, C73, C74, C75, C76, C77, C78, C79, C8, C80, C81, C82, C83, C86, C87, C88, C89, C9, C90, C91, C92, C93, C94, C97, C98, C99: value (none) -> 10n
- C100, C105, C108, C111, C115, C35, C46, C5, C51, C52, C7, C95, C96: value (none) -> 100n
- C103, C109, C113, C16, C38, C4, C84: value (none) -> 10u 0805
- C104, C85: value (none) -> 22u 0805
- C106: value (none) -> 22p
- C107, C112: value (none) -> 4u7 0603
- C110, C23, C32, C55, C57, C6, LED2, R103, R104, R113, R63, R93, R98: value (none) -> NP
- C114, C37, C45: value (none) -> 1n 1206
- C119, C3: value (none) -> 1u 0603
- C18, C19, C25, C28, C48, C49, C50, C53, C60, C61: value (none) -> 12p
- C20, C21: value (none) -> 1p2
- C22, C26, C33, C34: value (none) -> 2p4
- C24: value (none) -> 10p
- C27: value (none) -> 1p6
- C29: value (none) -> 0n
- C30, L2, L3, L4, L5, L6, L7, L8, L9: value (none) -> low ind
- C31: value (none) -> 0p5
- C36, L11, R76, R77, R78, R79: value (none) -> 50R
- C62: value (none) -> 100p
- L1, R101, R102, R106, R107, R112, R16, R18, R96, R97: value (none) -> 0R
- L13: value (none) -> 1u
- L14: value (none) -> 4u
- LED3: value (none) -> Blue LED
- Q1, Q2: value (none) -> S8550M
- R100: value (none) -> 66k4
- R108, R109, R57, R91: value (none) -> 1k
- R11, R12, R13, R14, R15, R17, R2, R3, R4, R52, R53, R58, R62, R82, R84: value (none) -> 10k
- R110, R111, R60, R92: value (none) -> 3k
- R20: value (none) -> 2k4
- R21, R22, R23, R24, R25, R26, R27, R28, R29, R30, R31, R32, R33, R34, R35, R36, R37, R38, R39, R40, R41, R42, R43, R44, R45, R46, R47, R48, R49, R50, R51, R54, R56: value (none) -> 22R
- R55: value (none) -> 100R; device TL-WR703N:C0402 -> TL-WR703N:R0402
- R59, R61, R7: value (none) -> 6k2
- R64, R65, R68, R71: value (none) -> 75R
- R83: value (none) -> 3k8
- R94: value (none) -> 0R 0603
- R95: value (none) -> 10R 0603
- R99: value (none) -> 299k; device TL-WR703N:C0402 -> TL-WR703N:R0402
- U3: value (none) -> S25FL032P0XMFI01
- Y1: value (none) -> 25.00 MHz
- renumbered E$9 to GND_CONTACTS, R6 to R61
Connections:
- net S$1 renamed A3_B
- net S$10 renamed A4_B
- net S$104 renamed D-
- net S$105 renamed GPIO11
- net S$108 renamed +5V0
- net S$11 renamed A5_B
- net S$113 renamed USB_POWER
- net S$118 renamed LX
- net S$119 renamed XOUT
- net S$12 renamed A8_B
- net S$120 renamed +1V2
- net S$126 renamed FB
- net S$13 renamed A9_B
- net S$132 renamed +2V5
- net S$14 renamed A12_B
- net S$147 renamed GPIO6
- net S$148 renamed USB_DP
- net S$150 renamed GPIO7
- net S$157 renamed TX_GND
- net S$159 renamed !SPI_W
- net S$16 renamed DQ0_B
- net S$161 renamed N$3
- net S$162 renamed RX+
- net S$165 renamed !SPI_CS_0
- net S$171 renamed GPIO1
- net S$172 renamed DQ9_B
- net S$178 renamed ANT1_INT
- net S$180 renamed SPI_CLK
- net S$182 renamed D+
- net S$19 renamed CKE
- net S$193 renamed ETH_GND
- net S$199 renamed SPI_SO
- net S$2 renamed A2_B
- net S$20 renamed A2
- net S$21 renamed A0
- net S$22 renamed DQ1_B
- net S$221 renamed N$4
- net S$224 renamed +2V0
- net S$228 renamed LDO
- net S$23 renamed DQ2_B
- net S$238 renamed LED3
- net S$239 renamed +3V3
- net S$24 renamed DQ3_B
- net S$25 renamed DQ4B
- net S$252 renamed TX+
- net S$26 renamed DQ5_B
- net S$269 renamed VBUS
- net S$27 renamed DQ6_B
- net S$28 renamed TD-
- net S$29 renamed RX-
- net S$3 renamed A1_B
- net S$30 renamed DQ7_B
- net S$31 renamed LDQS_B
- net S$32 renamed DQ0
- net S$33 renamed DQ1
- net S$34 renamed DQ2
- net S$344 renamed UDM
- net S$345 renamed DQ8_B
- net S$346 renamed DQ10_B
- net S$347 renamed DQ12_B
- net S$348 renamed DQ14_B
- net S$349 renamed DQ15_B
- net S$35 renamed DQ3
- net S$350 renamed DQ13_B
- net S$351 renamed DQ11_B
- net S$361 renamed DQ11
- net S$362 renamed DQ12
- net S$363 renamed DQ9
- net S$364 renamed DQ10
- net S$366 renamed UDQS
- net S$369 renamed UDQS_B
- net S$37 renamed DQ5
- net S$371 renamed TD+
- net S$373 renamed RD-
- net S$375 renamed !CAS
- net S$376 renamed !WE
- net S$377 renamed !RAS
- net S$378 renamed !CS
- net S$38 renamed DQ6
- net S$382 renamed BA0
- net S$383 renamed BA1
- net S$39 renamed DQ7
- net S$4 renamed A0_B
- net S$40 renamed LDQS
- net S$41 renamed TX-
- net S$416 renamed DQ15
- net S$42 renamed RX_GND
- net S$420 renamed DQ8
- net S$428 renamed DQ14
- net S$429 renamed DQ13
- net S$43 renamed !CLK
- net S$431 renamed DQ4
- net S$449 renamed GPIO29
- net S$46 renamed CLK
- net S$47 renamed GPIO0
- net S$5 renamed A10_B/AP_B
- net S$51 renamed GPIO17
- net S$52 renamed GPIO14
- net S$53 renamed !CLK_B
- net S$56 renamed LDM
- net S$57 renamed A3
- net S$58 renamed A1
- net S$59 renamed A10/AP
- net S$6 renamed TP_OUT
- net S$60 renamed CLK_B
- net S$61 renamed A11
- net S$62 renamed A8
- net S$63 renamed A6
- net S$64 renamed A5
- net S$65 renamed A7
- net S$66 renamed A9
- net S$7 renamed A11_B
- net S$71 renamed RD+
- net S$74 renamed A4
- net S$77 renamed GPIO13
- net S$79 renamed SPI_MISO
- net S$8 renamed A7_B
- net S$83 renamed ANT1
- net S$84 renamed A12
- net S$86 renamed TP_IN
- net S$88 renamed GPIO15
- net S$89 renamed XIN
- net S$9 renamed A6_B
- net S$96 renamed SPI_MOSI
- net S$97 renamed GPIO8
- net S$98 renamed USB_DM
- net S$99 renamed GPIO16
- removed net S$292: C37.2, C45.1, J3.S$2
- removed net S$85: C48.1, C52.1
- new net N$1: C79.1, U1.A71
- net GND: now also C48.1, C52.1
- net S$18: no longer C79.1, U1.A71
- net SHIELD: now also C37.2, C45.1, J3.S$2
Routing:
- net SHIELD: track 39.6 -> 53.8 mm, vias 0 -> 1
- net S$292: track 14.3 -> 0.00 mm, vias 1 -> 0
- net S$18: track 38.9 -> 36.5 mm, vias 4 -> 3
- net N$1: track 0.00 -> 1.45 mm, vias 0 -> 1
- net S$85: track 1.04 -> 0.00 mm
- net GND: track 37.1 -> 38.2 mm
- net N$4: track 1.46 -> 1.08 mm, vias 1 -> 0
- net D+: vias 2 -> 1
- net +2V0: vias 4 -> 3
Other:
- board text added: "0"
- board text added: "1"
- board text added: "2"
- board text added: "3"
- board text added: "4"
- board text added: "5"
- board text added: "6"
- board text added: "7"
- board text added: "8"
- board text added: "9"
- board text added: "A"
- board text added: "B"
- board text added: "C"
- board text added: "D"
- board text added: "E"
- board text added: "F"
- board text added: "G"
- board text added: "H"
- board text added: "I"
- board text added: "J"
- board text added: "K"
- board text added: "L"
- board text added: "M"
- board text added: "N"
- board text added: "O"
- board text added: "P"
- board text added: "Q"
- board text added: "http://squonk42.github.com/TL-WR703N/"
- board text removed: "®"
