File: CAD/TL-WR703N.sch (EAGLE design)
At the start: 241 parts, among them J1 JUMPER, J3 RJ45_2SH, Q1 S8550M, Q2 S8550M, SW2 TACT_SWITCH_SPST, T1 ETH10_100_TRANSFO, U1 AR9331-AL1A, U2 A3S56F40FTP, U3 S25FL032P0XMFI01, U5 UNKNOWN_BUCK, U6 TPS2041BDBV, Y1 25.00 MHz

Commit message: Updated board to Rev. B
Added missing wire between c21 and C28, and between U1-A33 and +2V5.
Removed internal via labels after probing with a DMM
Connections:
- net S$156 renamed ANT1_OUTN
- net S$50 renamed ANT1_INN
- net S$68 renamed ANT1_INP
- net S$75 renamed ANT1_OUTP
- removed net N$3: D1.C
- removed net N$4: D2.C
- removed net S$112: L2.1
- removed net S$123: U1.A33
- removed net S$142: R97.2
- removed net S$143: R96.2
- removed net S$154: R95.1
- removed net S$164: R91.1
- removed net S$190: R62.1
- removed net S$216: C70.2, Q1.E, R93.2
- removed net S$230: R83.1
- removed net S$265: R108.2, R109.1
- removed net S$294: LED2.A, LED3.A
- removed net S$329: C92.2, R106.2, R98.2
- removed net S$359: C103.1, Q2.C, TPDDR.PP
- removed net S$372: C52.2, R78.1
- removed net S$390: R59.1
- removed net S$415: C4.2
- removed net S$45: C38.2
- removed net S$67: C18.1, C24.1, C85.2, L4.2
- removed net S$72: R82.1
- removed net S$81: C27.1, C28.1
- removed net S$82: R14.2, R2.1, R3.1
- removed net S$93: C7.1, U3.VCC
- removed net VDDQ: C11.2, C12.2, C15.1, C8.1, C9.2, U2.VDDQ@0, U2.VDDQ@1, U2.VDDQ@2, U2.VDDQ@3, U2.VDDQ@4
- net $28: now also C52.2, R78.1
- net +2V5: now also R14.2, R2.1, R3.1, R82.1, U1.A33
- net +3V3: now also C18.1, C24.1, C38.2, C4.2, C7.1, C70.2, C85.2, C92.2, D1.C, D2.C, L2.1, L4.2, LED2.A, LED3.A, Q1.E, R106.2, R108.2, R109.1, R62.1, R91.1, R93.2, R95.1, R96.2, R97.2, R98.2, U3.VCC
- net LED3: now also R83.1
- net S$80: now also C27.1, C28.1
- net VDD: now also C103.1, C11.2, C12.2, C15.1, C8.1, C9.2, Q2.C, R59.1, TPDDR.PP, U2.VDDQ@0, U2.VDDQ@1, U2.VDDQ@2, U2.VDDQ@3, U2.VDDQ@4
Other:
- note added: "Rev. B"
- note removed: "0"
- note removed: "1"
- note removed: "2"
- note removed: "3"
- note removed: "4"
- note removed: "5"
- note removed: "6"
- note removed: "7"
- note removed: "8"
- note removed: "9"
- note removed: "A"
- note removed: "B"
- note removed: "C"
- note removed: "D"
- note removed: "E"
- note removed: "F"
- note removed: "G"
- note removed: "H"
- note removed: "I"
- note removed: "J"
- note removed: "K"
- note removed: "M"
- note removed: "N"
- note removed: "O"
- note removed: "P"
- note removed: "Q"
- note removed: "Rev. A"
- moved on the sheet: C15, C16, C17, C18, C24, C4, C6, C8, C85, R55, R59, R61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
